Commit message: edit: joint limits in full body URDF

File: source/isaaclab_assets/data/Hanu/full_body_description/urdf/full_body.urdf (robot description, URDF)
Before this commit: robot full_body, 34 links, 33 joints
Joints:
- joint torso to abdomen Yaw: limit effort=32 velocity=20 -> lower=-1.5708 upper=1.5708 effort=32 velocity=20
