Commit message: edit: usd path for 4090

File: source/isaaclab_assets/data/Robots/hanu/hanumanoid_description/urdf/hanumanoid.urdf (robot description, URDF)
Before this commit: robot hanumanoid, 37 links, 36 joints
Links:
- link E1R_1: geometry collision mesh filename=/home/ubuntu/IsaacLab/source/isaaclab_assets/data/Robots/ha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 scale=0.001 0.001 0.001; visual mesh filename=/home/ubuntu/IsaacLab/source/isaaclab_assets/data/Robots/ha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 scale=0.001 0.001 0.001
- link abdomen_1: geometry collision mesh filename=/home/ubuntu/IsaacLab/source/isaaclab_assets/data/Robots/ha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 scale=0.001 0.001 0.001; visual mesh filename=/home/ubuntu/IsaacLab/source/isaaclab_assets/data/Robots/ha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 scale=0.001 0.001 0.001
- link base_link: geometry collision mesh filename=/home/ubuntu/IsaacLab/source/isaaclab_assets/data/Robots/ha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 scale=0.001 0.001 0.001; visual mesh filename=/home/ubuntu/IsaacLab/source/isaaclab_assets/data/Robots/ha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 scale=0.001 0.001 0.001
- link fixed_imu_1: geometry collision mesh filename=/home/ubuntu/IsaacLab/source/isaaclab_assets/data/Robots/ha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 scale=0.001 0.001 0.001; visual mesh filename=/home/ubuntu/IsaacLab/source/isaaclab_assets/data/Robots/ha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 scale=0.001 0.001 0.001
- link fixed_mid_360_1: geometry collision mesh filename=/home/ubuntu/IsaacLab/source/isaaclab_assets/data/Robots/ha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 scale=0.001 0.001 0.001; visual mesh filename=/home/ubuntu/IsaacLab/source/isaaclab_assets/data/Robots/ha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 scale=0.001 0.001 0.001
- link l_ankle_pitch_1: geometry collision mesh filename=/home/ubuntu/IsaacLab/source/isaaclab_assets/data/Robots/ha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 scale=0.001 0.001 0.001; visual mesh filename=/home/ubuntu/IsaacLab/source/isaaclab_assets/data/Robots/ha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 scale=0.001 0.001 0.001
- link l_calf_pitch_1: geometry collision mesh filename=/home/ubuntu/IsaacLab/source/isaaclab_assets/data/Robots/ha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 scale=0.001 0.001 0.001; visual mesh filename=/home/ubuntu/IsaacLab/source/isaaclab_assets/data/Robots/ha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 scale=0.001 0.001 0.001
- link l_contact_sensor_1: geometry collision mesh filename=/home/ubuntu/IsaacLab/source/isaaclab_assets/data/Robots/ha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 scale=0.001 0.001 0.001; visual mesh filename=/home/ubuntu/IsaacLab/source/isaaclab_assets/data/Robots/ha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 scale=0.001 0.001 0.001
- link l_foot_pressure_sensor_1: geometry collision mesh filename=/home/ubuntu/IsaacLab/source/isaaclab_assets/data/Robots/ha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 scale=0.001 0.001 0.001; visual mesh filename=/home/ubuntu/IsaacLab/source/isaaclab_assets/data/Robots/ha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 scale=0.001 0.001 0.001
- link l_foot_roll_1: geometry collision mesh filename=/home/ubuntu/IsaacLab/source/isaaclab_assets/data/Robots/ha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 scale=0.001 0.001 0.001; visual mesh filename=/home/ubuntu/IsaacLab/source/isaaclab_assets/data/Robots/ha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 scale=0.001 0.001 0.001
- link l_glute_pitch_1: geometry collision mesh filename=/home/ubuntu/IsaacLab/source/isaaclab_assets/data/Robots/ha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 scale=0.001 0.001 0.001; visual mesh filename=/home/ubuntu/IsaacLab/source/isaaclab_assets/data/Robots/ha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 scale=0.001 0.001 0.001
- link l_groin_yaw_1: geometry collision mesh filename=/home/ubuntu/IsaacLab/source/isaaclab_assets/data/Robots/ha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 scale=0.001 0.001 0.001; visual mesh filename=/home/ubuntu/IsaacLab/source/isaaclab_assets/data/Robots/ha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 scale=0.001 0.001 0.001
- link l_hand_roll_1: geometry collision mesh filename=/home/ubuntu/IsaacLab/source/isaaclab_assets/data/Robots/ha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 scale=0.001 0.001 0.001; visual mesh filename=/home/ubuntu/IsaacLab/source/isaaclab_assets/data/Robots/ha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 scale=0.001 0.001 0.001
- link l_lowerarm_pitch_1: geometry collision mesh filename=/home/ubuntu/IsaacLab/source/isaaclab_assets/data/Robots/ha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 scale=0.001 0.001 0.001; visual mesh filename=/home/ubuntu/IsaacLab/source/isaaclab_assets/data/Robots/ha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 scale=0.001 0.001 0.001
- link l_shoulder_pitch_1: geometry collision mesh filename=/home/ubuntu/IsaacLab/source/isaaclab_assets/data/Robots/ha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 scale=0.001 0.001 0.001; visual mesh filename=/home/ubuntu/IsaacLab/source/isaaclab_assets/data/Robots/ha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 scale=0.001 0.001 0.001
- link l_shoulder_roll_1: geometry collision mesh filename=/home/ubuntu/IsaacLab/source/isaaclab_assets/data/Robots/ha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 scale=0.001 0.001 0.001; visual mesh filename=/home/ubuntu/IsaacLab/source/isaaclab_assets/data/Robots/ha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 scale=0.001 0.001 0.001
- link l_thigh_roll_1: geometry collision mesh filename=/home/ubuntu/IsaacLab/source/isaaclab_assets/data/Robots/ha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 scale=0.001 0.001 0.001; visual mesh filename=/home/ubuntu/IsaacLab/source/isaaclab_assets/data/Robots/ha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 scale=0.001 0.001 0.001
- link l_upperarm_yaw_1: geometry collision mesh filename=/home/ubuntu/IsaacLab/source/isaaclab_assets/data/Robots/ha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 scale=0.001 0.001 0.001; visual mesh filename=/home/ubuntu/IsaacLab/source/isaaclab_assets/data/Robots/ha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 scale=0.001 0.001 0.001
- link l_wrist_pitch_1: geometry collision mesh filename=/home/ubuntu/IsaacLab/source/isaaclab_assets/data/Robots/ha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 scale=0.001 0.001 0.001; visual mesh filename=/home/ubuntu/IsaacLab/source/isaaclab_assets/data/Robots/ha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 scale=0.001 0.001 0.001
- link l_wrist_yaw_1: geometry collision mesh filename=/home/ubuntu/IsaacLab/source/isaaclab_assets/data/Robots/ha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 scale=0.001 0.001 0.001; visual mesh filename=/home/ubuntu/IsaacLab/source/isaaclab_assets/data/Robots/ha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 scale=0.001 0.001 0.001
- link neck_1: geometry collision mesh filename=/home/ubuntu/IsaacLab/source/isaaclab_assets/data/Robots/ha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 scale=0.001 0.001 0.001; visual mesh filename=/home/ubuntu/IsaacLab/source/isaaclab_assets/data/Robots/ha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 scale=0.001 0.001 0.001
- link r_ankle_pitch_1: geometry collision mesh filename=/home/ubuntu/IsaacLab/source/isaaclab_assets/data/Robots/ha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 scale=0.001 0.001 0.001; visual mesh filename=/home/ubuntu/IsaacLab/source/isaaclab_assets/data/Robots/ha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 scale=0.001 0.001 0.001
- link r_calf_pitch_1: geometry collision mesh filename=/home/ubuntu/IsaacLab/source/isaaclab_assets/data/Robots/ha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 scale=0.001 0.001 0.001; visual mesh filename=/home/ubuntu/IsaacLab/source/isaaclab_assets/data/Robots/ha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 scale=0.001 0.001 0.001
- link r_contact_sensor_1: geometry collision mesh filename=/home/ubuntu/IsaacLab/source/isaaclab_assets/data/Robots/ha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 scale=0.001 0.001 0.001; visual mesh filename=/home/ubuntu/IsaacLab/source/isaaclab_assets/data/Robots/ha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 scale=0.001 0.001 0.001
- link r_foot_pressure_sensor_1: geometry collision mesh filename=/home/ubuntu/IsaacLab/source/isaaclab_assets/data/Robots/ha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 scale=0.001 0.001 0.001; visual mesh filename=/home/ubuntu/IsaacLab/source/isaaclab_assets/data/Robots/ha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 scale=0.001 0.001 0.001
- link r_foot_roll_1: geometry collision mesh filename=/home/ubuntu/IsaacLab/source/isaaclab_assets/data/Robots/ha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 scale=0.001 0.001 0.001; visual mesh filename=/home/ubuntu/IsaacLab/source/isaaclab_assets/data/Robots/ha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 scale=0.001 0.001 0.001
- link r_glute_pitch_1: geometry collision mesh filename=/home/ubuntu/IsaacLab/source/isaaclab_assets/data/Robots/ha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 scale=0.001 0.001 0.001; visual mesh filename=/home/ubuntu/IsaacLab/source/isaaclab_assets/data/Robots/ha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 scale=0.001 0.001 0.001
- link r_groin_yaw_1: geometry collision mesh filename=/home/ubuntu/IsaacLab/source/isaaclab_assets/data/Robots/ha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 scale=0.001 0.001 0.001; visual mesh filename=/home/ubuntu/IsaacLab/source/isaaclab_assets/data/Robots/ha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 scale=0.001 0.001 0.001
- link r_hand_roll_1: geometry collision mesh filename=/home/ubuntu/IsaacLab/source/isaaclab_assets/data/Robots/ha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 scale=0.001 0.001 0.001; visual mesh filename=/home/ubuntu/IsaacLab/source/isaaclab_assets/data/Robots/ha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 scale=0.001 0.001 0.001
- link r_lowerarm_pitch_1: geometry collision mesh filename=/home/ubuntu/IsaacLab/source/isaaclab_assets/data/Robots/ha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 scale=0.001 0.001 0.001; visual mesh filename=/home/ubuntu/IsaacLab/source/isaaclab_assets/data/Robots/ha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 scale=0.001 0.001 0.001
- link r_shoulder_pitch_1: geometry collision mesh filename=/home/ubuntu/IsaacLab/source/isaaclab_assets/data/Robots/ha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 scale=0.001 0.001 0.001; visual mesh filename=/home/ubuntu/IsaacLab/source/isaaclab_assets/data/Robots/ha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 scale=0.001 0.001 0.001
- link r_shoulder_roll_1: geometry collision mesh filename=/home/ubuntu/IsaacLab/source/isaaclab_assets/data/Robots/ha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 scale=0.001 0.001 0.001; visual mesh filename=/home/ubuntu/IsaacLab/source/isaaclab_assets/data/Robots/ha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 scale=0.001 0.001 0.001
- link r_thigh_roll_1: geometry collision mesh filename=/home/ubuntu/IsaacLab/source/isaaclab_assets/data/Robots/ha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 scale=0.001 0.001 0.001; visual mesh filename=/home/ubuntu/IsaacLab/source/isaaclab_assets/data/Robots/ha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 scale=0.001 0.001 0.001
- link r_upperarm_yaw_1: geometry collision mesh filename=/home/ubuntu/IsaacLab/source/isaaclab_assets/data/Robots/ha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 scale=0.001 0.001 0.001; visual mesh filename=/home/ubuntu/IsaacLab/source/isaaclab_assets/data/Robots/ha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 scale=0.001 0.001 0.001
- link r_wrist_pitch_1: geometry collision mesh filename=/home/ubuntu/IsaacLab/source/isaaclab_assets/data/Robots/ha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 scale=0.001 0.001 0.001; visual mesh filename=/home/ubuntu/IsaacLab/source/isaaclab_assets/data/Robots/ha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 scale=0.001 0.001 0.001
- link r_wrist_yaw_1: geometry collision mesh filename=/home/ubuntu/IsaacLab/source/isaaclab_assets/data/Robots/ha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 scale=0.001 0.001 0.001; visual mesh filename=/home/ubuntu/IsaacLab/source/isaaclab_assets/data/Robots/ha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 scale=0.001 0.001 0.001
- link torso_1: geometry collision mesh filename=/home/ubuntu/IsaacLab/source/isaaclab_assets/data/Robots/ha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 scale=0.001 0.001 0.001; visual mesh filename=/home/ubuntu/IsaacLab/source/isaaclab_assets/data/Robots/ha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 scale=0.001 0.001 0.001
